Commit message: updated pybullet demos

File: manipulator_env/models/ur10e_robotiq85.urdf (robot description, URDF)
Before this commit: robot ur10e_robotiq85, 19 links, 18 joints
Links:
- link forearm_link: mass 3.989 -> 3.87
- link shoulder_link: mass 7.369 -> 7.778
- link upper_arm_link: mass 13.051 -> 12.93
- link wrist_1_link: mass 2.1 -> 1.96
- link wrist_2_link: mass 1.98 -> 1.96
- link wrist_3_link: mass 0.615 -> 0.202
Joints:
- joint wrist_1_joint: limit lower=-6.283185307179586 upper=6.283185307179586 effort=54.0 velocity=3.141592653589793 -> lower=-6.283185307179586 upper=6.283185307179586 effort=56.0 velocity=3.141592653589793
- joint wrist_2_joint: limit lower=-6.283185307179586 upper=6.283185307179586 effort=54.0 velocity=3.141592653589793 -> lower=-6.283185307179586 upper=6.283185307179586 effort=56.0 velocity=3.141592653589793

Commit message: updated base and griper offset results same as of real robot

File: manipulator_env/models/ur10e_robotiq85.urdf (robot description, URDF)
Before this commit: robot ur10e_robotiq85, 19 links, 18 joints
Links:
- added link base
- link base_link: mass 0.0 -> None
- link flange: mass 0.0 -> None
- link tool0: mass 0.0 -> None
Joints:
- removed joint finger_joint
- added joint base_link-base_fixed_joint: type fixed, parent base_link, child base, origin xyz=0 0 0 rpy=0 0 3.141592653589793
- added joint robotiq_85_left_knuckle_joint: type revolute, parent robotiq_85_base_link, child robotiq_85_left_knuckle_link, origin xyz=0.05490451627 0.03060114443 0.0 rpy=3.141592653589793 0.0 0.0, axis 0 0 1, limit lower=0.0 upper=0.80285 effort=1000 velocity=0.5
- joint robotiq_85_base_joint: origin xyz=0 0 0 rpy=0 -1.5707963267948966 0 -> xyz=0 0 0 rpy=0 -1.57079632679 1.57079632679
- joint robotiq_85_left_finger_tip_joint: mimic joint=finger_joint multiplier=-1 offset=0 -> joint=robotiq_85_left_knuckle_joint multiplier=-1; type revolute -> continuous
- joint robotiq_85_left_inner_knuckle_joint: mimic joint=finger_joint multiplier=1 offset=0 -> joint=robotiq_85_left_knuckle_joint offset=0; type revolute -> continuous
- joint robotiq_85_right_finger_tip_joint: mimic joint=finger_joint multiplier=-1 offset=0 -> joint=robotiq_85_left_knuckle_joint multiplier=-1; origin xyz=0.04303959807 -0.03759940821 0.0 rpy=0.0 0.0 0.0 -> xyz=0.04303959807 -0.03759940821  0.0 rpy=0.0 0.0 0.0; type revolute -> continuous
- joint robotiq_85_right_inner_knuckle_joint: mimic joint=finger_joint multiplier=1 offset=0 -> joint=robotiq_85_left_knuckle_joint offset=0; type revolute -> continuous
- joint robotiq_85_right_knuckle_joint: limit lower=0.0 upper=0.80285 effort=1000 velocity=0.5 -> lower=-3.14 upper=3.14 effort=1000 velocity=100.0; mimic joint=finger_joint multiplier=1 offset=0 -> joint=robotiq_85_left_knuckle_joint; type revolute -> continuous
- joint wrist_2_joint: origin xyz=0 -0.11985 0 rpy=1.570796327 0 0 -> xyz=0 -0.11985 -2.458164590756244e-11 rpy=1.570796327 0 0
- joint wrist_3_joint: limit lower=-6.283185307179586 upper=6.283185307179586 effort=54.0 velocity=3.141592653589793 -> lower=-6.283185307179586 upper=6.283185307179586 effort=56.0 velocity=3.141592653589793; origin xyz=0 0.11655 0 rpy=1.570796326589793 3.141592653589793 3.141592653589793 -> xyz=0 0.11655 -2.390480459346185e-11 rpy=1.570796326589793 3.141592653589793 3.141592653589793
